Commit message: 2

File: src/amr/urdf/amr_robot.urdf (robot description, URDF)
Before this commit: robot amr_robot, 9 links, 8 joints
Links:
- link arm_base_link: mass None -> 0.1
- link arm_link: mass None -> 0.2
- link base_link: mass 5.0 -> 2.0; geometry collision box size=0.3 0.2 0.06; visual box size=0.4 0.3 0.1
- link camera_link: mass None -> 0.05
- link caster_wheel: mass 0.2 -> 0.1
- link laser_link: mass None -> 0.1
- link left_wheel: mass 0.5 -> 0.2
- link right_wheel: mass 0.5 -> 0.2
Joints:
- joint arm_pivot_joint: child  -> arm_base_link
- joint base_joint: origin xyz=0 0 0.05 -> xyz=0 0 0.08
- joint caster_joint: origin xyz=0.15 0 -0.01 -> xyz=0.15 0 -0.03
- joint left_wheel_joint: origin xyz=-0.1 0.17 0 rpy=-1.57 0 0 -> xyz=-0.1 0.17 -0.03 rpy=-1.5708 0 0
- joint right_wheel_joint: origin xyz=-0.1 -0.17 0 rpy=-1.57 0 0 -> xyz=-0.1 -0.17 -0.03 rpy=-1.5708 0 0

Commit message: 3

File: src/amr/urdf/amr_robot.urdf (robot description, URDF)
Before this commit: robot amr_robot, 9 links, 8 joints
Links:
- removed link arm_base_link
- removed link arm_link
- removed link camera_link
- link base_link: geometry collision box size=0.4 0.3 0.1; visual box size=0.4 0.3 0.1
Joints:
- removed joint arm_lift_joint
- removed joint arm_pivot_joint
- removed joint camera_joint

Commit message: fix: rviz小车大幅漂移

File: src/amr/urdf/amr_robot.urdf (robot description, URDF)
Before this commit: robot amr_robot, 6 links, 5 joints
Joints:
- joint laser_joint: origin xyz=0.1 0 0.07 -> xyz=0.1 0 0.07 rpy=0 0 0

Commit message: 多任务调度&充电

File: src/amr/urdf/amr_robot.urdf (robot description, URDF)
Before this commit: robot amr_robot, 6 links, 5 joints
Links:
- added link camera_link, mass 0.05; visual box size=0.04 0.06 0.04
Joints:
- added joint camera_joint: type fixed, parent base_link, child camera_link, origin xyz=0.22 0 0.12 rpy=0 0 0
